File: echoear_baseboard/echoear_baseboard.kicad_pcb (KiCad board)
At the start: 4 copper layers, 37.3 x 30.3 mm, 61 parts, among them Q1 AO3401A, Q2 AO3401A, SW1 TS-1088-AR02016, SW2 TS-1088-AR02016, SW3 TS-1088-AR02016, U1 TYPE-C 16PIN 2MD(073), U2 YZ92015035T-04025-01, U3 MountingHole_Pad, U4 A-SP1102DR6GHC-C01-2C, U5 MountingHole_Pad, U6 TLV62569DBV, U7 TP4057, U8 SAM8108

Commit message: Updated prod files
Parts:
- turned U2 to 180 degrees
Routing:
- net GND: track 14.8 -> 13.8 mm
- net /VBUS: track 52.7 -> 53.8 mm
