File: echoear_baseboard/echoear_baseboard.kicad_sch (KiCad schematic)
At the start: 59 parts, among them Q1 AO3401A, Q2 AO3401A, SW1 TS-1088-AR02016, SW2 TS-1088-AR02016, SW3 TS-1088-AR02016, U1 TYPE-C 16PIN 2MD(073), U2 YZ92015035T-04025-01, U3 MountingHole_Pad, U4 A-SP1102DR6GHC-C01-2C, U5 MountingHole_Pad, U6 TLV62569DBV, U7 TP4057, U8 SAM8108

Commit message: Current echoear baseboard
Parts:
- D2, D3, D4: LCSC C383211 -> C5246195
Changed lines of the file:
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@@
 			)
 		)
-		(property "Description" "Bidirectional ESD protection diode, ±5.5Vrwm, 0.23pF, SG-WLL-2-3"
+		(property "Description" "100W@8/20us 12V 15pF 1uA 5.5V 5V ESD IEC 61000-4-2、IEC 61000-4-5、IEC 61000-4-4 SOD-523 ESD and Surge Protection (TVS/ESD) ROHS"
 			(at 208.28 48.26 0)
 			(hide yes)
@@
 			)
 		)
-		(property "LCSC" "C383211"
+		(property "LCSC" "C5246195"
 			(at 208.28 48.26 90)
 			(hide yes)
@@
 			)
 		)
-		(property "Description" "Bidirectional ESD protection diode, ±5.5Vrwm, 0.23pF, SG-WLL-2-3"
+		(property "Description" "100W@8/20us 12V 15pF 1uA 5.5V 5V ESD IEC 61000-4-2、IEC 61000-4-5、IEC 61000-4-4 SOD-523 ESD and Surge Protection (TVS/ESD) ROHS"
 			(at 257.81 54.61 0)
 			(hide yes)
@@
 			)
 		)
-		(property "LCSC" "C383211"
+		(property "LCSC" "C5246195"
 			(at 257.81 54.61 90)
 			(hide yes)
@@
 			)
 		)
-		(property "Description" "Bidirectional ESD protection diode, ±5.5Vrwm, 0.23pF, SG-WLL-2-3"
+		(property "Description" "100W@8/20us 12V 15pF 1uA 5.5V 5V ESD IEC 61000-4-2、IEC 61000-4-5、IEC 61000-4-4 SOD-523 ESD and Surge Protection (TVS/ESD) ROHS"
 			(at 254 54.61 0)
 			(hide yes)
@@
 			)
 		)
-		(property "LCSC" "C383211"
+		(property "LCSC" "C5246195"
 			(at 254 54.61 90)
 			(hide yes)

Commit message: Updated prod files
Parts:
- R12: LCSC C26082 -> C2933065
Changed lines of the file:
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@@
 			)
 		)
-		(property "LCSC" "C26082"
+		(property "LCSC" "C2933065"
 			(at 109.22 114.3 0)
 			(hide yes)
