File: echoear_coreboard/codec1.kicad_sch (KiCad schematic)
At the start: 36 parts, among them Q3 LBSS138DW1T1G, Q4 LBSS138DW1T1G, U4 XC6206P332MR, U6 ES8311

Commit message: Finished coreboard SCH w/o ERC check
Parts:
- removed C10: 2.2n, Capacitor_SMD:C_0402_1005Metric, symbol Device:C
- removed C11: 100p, Capacitor_SMD:C_0402_1005Metric, symbol Device:C
- removed C12, C13, C16, C24, C25, C27, C29, C30, C32: 1u, Capacitor_SMD:C_0402_1005Metric, symbol Device:C
- removed C14, C7: 470n, Capacitor_SMD:C_0402_1005Metric, symbol Device:C
- removed C15, C8: 220n, Capacitor_SMD:C_0402_1005Metric, symbol Device:C
- removed C31: 100n, Capacitor_SMD:C_0402_1005Metric, symbol Device:C
- removed C33, C34, C39, C40, C41: 22p, Capacitor_SMD:C_0402_1005Metric, symbol Device:C
- removed C9: 10n, Capacitor_SMD:C_0402_1005Metric, symbol Device:C
- removed Q3, Q4: LBSS138DW1T1G, easyeda2kicad:SC-88-6_L2.0-W1.3-P0.65-LS2.1-BL, symbol Sym_easyeda2kicad:LBSS138DW1T1G
- removed R10: 4.3k, Capacitor_SMD:C_0402_1005Metric, symbol Device:R
- removed R11, R15, R6, R7: 2.2k, Resistor_SMD:R_0402_1005Metric, symbol Device:R
- removed R12, R8: 10k, Resistor_SMD:R_0402_1005Metric, symbol Device:R
- removed R13: 20k, Capacitor_SMD:C_0402_1005Metric, symbol Device:R
- removed R14: 0R, Resistor_SMD:R_0402_1005Metric, symbol Device:R
- removed R9: 20k, Resistor_SMD:R_0402_1005Metric, symbol Device:R
- removed U4: XC6206P332MR, easyeda2kicad:SOT-23-3_L2.9-W1.6-P1.90-LS2.8-BR, symbol Sym_easyeda2kicad:XC6206P332MR
- removed U6: ES8311, easyeda2kicad:WQFN-20_L3.0-W3.0-P0.40-BL-EP1.7, symbol Sym_easyeda2kicad:ES8311
- added C42, C43: 1n, Capacitor_SMD:C_0402_1005Metric, symbol Device:C
- added C44, C45, C53: 100n, Capacitor_SMD:C_0402_1005Metric, symbol Device:C
- added C46, C49, C52, C54, C55, C56, C57, C58, C59, C60, C61, C62, C63, C64: 1u, Capacitor_SMD:C_0402_1005Metric, symbol Device:C
- added C47, C48: 22u, Capacitor_SMD:C_0603_1608Metric, symbol Device:C
- added CN4: HC-1.25-2PLT, easyeda2kicad:CONN-SMD_HC-1.25-2PLT, symbol Sym_easyeda2kicad:HC-1.25-2PLT
- added FPC2: AFC11-S08ICA-00, easyeda2kicad:CONN-TH-8P_AFC11-S08ICA-00, symbol Sym_easyeda2kicad:AFC11-S08ICA-00
- added R18, R24: 10k, Resistor_SMD:R_0402_1005Metric, symbol Device:R
- added R19, R20: 100k, Resistor_SMD:R_0402_1005Metric, symbol Device:R
- added R21: R, Resistor_SMD:R_0402_1005Metric, symbol Device:R
- added U7: NS4150, easyeda2kicad:MSOP-8_L3.0-W3.0-P0.65-LS5.0-BL, symbol Sym_easyeda2kicad:NS4150
- added U8: ES7210, easyeda2kicad:QFN-32_L4.0-W4.0-P0.40-BL-EP2.7, symbol Sym_easyeda2kicad:ES7210
Connections:
- net ADC_MIC3_N: now also U8.32 (MIC3N)
- net ADC_MIC3_P: now also U8.31 (MIC3P)
- net AUDIO_I2C_SCL: now also U8.4 (CCLK)
- net AUDIO_I2C_SDA: now also U8.3 (CDATA)
- net CODEC_3V3: now also C52.1, C53.2, C56.1, C64.1, U8.22 (VDDA), U8.23 (VDDM), U8.6 (VDDP), U8.7 (VDDD)
- net GND: now also C42.2, C43.2, C46.2, C47.2, C48.2, C49.2, CN4.3, CN4.4, FPC2.10, FPC2.9, R18.1, U7.7 (GND)
- net GNDA: now also C52.2, C53.1, C54.2, C55.2, C56.2, C57.2, C58.2, C59.2, C60.2, C61.2, C62.2, C63.2, C64.2, FPC2.6, R21.1, R24.1, U8.21 (GNDA), U8.33 (EP), U8.8 (GNDD)
- net I2S_BCK: now also U8.9 (SCLK)
- net I2S_MCLK: now also U8.5 (MCLK)
- net I2S_WS: now also U8.10 (LRCK)
- net MCU_3V3: now also FPC2.1
- net OUTN: now also C45.1
- net OUTP: now also C44.2
- new net: C58.1, U8.29 (REFP34)
- new net: R24.2, U8.1 (AD0)
- new net: C54.1, U8.17 (REFP12)
- new net: C55.1, U8.18 (REFQ12)
- new net: R21.2, U8.2 (AD1)
- new net: C62.1, U8.25 (REFQM)
- new net: C61.1, U8.26 (MICBIAS34)
- new net: C60.1, U8.27 (MIC4N)
- new net: C59.1, U8.28 (MIC4P)
- new net: C57.1, U8.30 (REFQ34)
- new net: C49.1, U7.2 (Bypass)
- new net: C45.2, R20.1
- new net: R20.2, U7.4 (INN)
- new net: R19.2, U7.3 (INP)
- new net: C44.1, R19.1
- new net ADC_MIC1_N: FPC2.8, U8.15 (MIC1N)
- new net ADC_MIC1_P: FPC2.7, U8.16 (MIC1P)
- new net ADC_MIC2_N: FPC2.4, U8.20 (MIC2N)
- new net ADC_MIC2_P: FPC2.5, U8.19 (MIC2P)
- new net ADC_MICBIAS12: C63.1, FPC2.3, U8.24 (MICBIAS12)
- new net I2S_DI: U8.11 (SDOUT1/TDMOUT)
- new net LED_G: FPC2.2
- new net PA_CTRL: R18.2, U7.1 (CTRL)
- new net VIN: C46.1, C47.1, C48.1, U7.6 (VCC)
- new net VON: C43.1, CN4.2, U7.5 (VON)
- new net VOP: C42.1, CN4.1, U7.8 (VoP)
Other:
- note added: "ES7210"
- note added: "MIC CONNECT"
- note added: "PA"
- note removed: "AEC"
- note removed: "CODEC 3V3 LDO"
- note removed: "CODEC_IIC"
- note removed: "ES8311"
