File: echoear_coreboard/echoear_coreboard.kicad_sch (KiCad schematic)
At the start: 4 parts, among them SW1 SW_SPST, U1 SAM8108, U2 TP4057

Commit message: Edited coreboard sch
Parts:
- removed R1: 4.7k, symbol Device:R
- removed SW1: SW_SPST, Button_Switch_SMD:SW-SMD_L3.9-W3.0-P4.45, symbol Switch:SW_SPST
- removed U1: SAM8108, Package_TO_SOT_SMD:SOT-23-6_L2.9-W1.6-P0.95-LS2.8-BL, symbol Driver_FET:LTC4440ES6
- removed U2: TP4057, Package_TO_SOT_SMD:SOT-23-6_L2.9-W1.6-P0.95-LS2.8-BL, symbol Driver_FET:LTC4440ES6
Connections:
- no-connect marks 2 -> 0
Other:
- note removed: "BAT CHARGE"
- note removed: "POWER ON/OFF MANAGEMENT"
- note removed: "PWR_EN"

Commit message: Setup and updated MCU schematic
Other:
- added sheet Interface (Interface.kicad_sch)
- added sheet MCU (MCU.kicad_sch)
- added sheet codec (codec.kicad_sch)
- note added: "SCH-ESP-VoCat-CoreBoard-V1_0"
Changed lines of the file:
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@@
 	(generator_version "10.0")
 	(paper "A4")
+	(text "SCH-ESP-VoCat-CoreBoard-V1_0"
+		(exclude_from_sim no)
+		(at 219.456 175.26 0)
+		(effects
+			(font
+				(size 3 3)
+				(thickness 0.6)
+				(bold yes)
+			)
+		)
+	)
+	(sheet
+		(at 185.42 92.71)
+		(size 26.67 13.97)
+		(exclude_from_sim no)
+		(in_bom yes)
+		(on_board yes)
+		(dnp no)
+		(fields_autoplaced yes)
+		(stroke
+			(width 0.1524)
+			(type solid)
+		)
+		(fill
+			(color 0 0 0 0)
+		)
+		(property "Sheetname" "codec"
+			(at 185.42 91.9984 0)
+			(show_name no)
+			(do_not_autoplace no)
+			(effects
+				(font
+					(size 1.27 1.27)
+				)
+				(justify left bottom)
+			)
+		)
+		(property "Sheetfile" "codec.kicad_sch"
+			(at 185.42 107.2646 0)
+			(show_name no)
+			(do_not_autoplace no)
+			(effects
+				(font
+					(size 1.27 1.27)
+				)
+				(justify left top)
+			)
+		)
+		(instances
+			(project "echoear_coreboard"
+				(path "/919b249b-28e6-49d6-a46c-47b0cfe0d5d1"
+					(page "4")
+				)
+			)
+		)
+	)
+	(sheet
+		(at 125.73 91.44)
+		(size 24.13 13.97)
+		(exclude_from_sim no)
+		(in_bom yes)
+		(on_board yes)
+		(dnp no)
+		(fields_autoplaced yes)
+		(stroke
+			(width 0.1524)
+			(type solid)
+		)
+		(fill
+			(color 0 0 0 0)
+		)
+		(property "Sheetname" "Interface"
+			(at 125.73 90.7284 0)
+			(show_name no)
+			(do_not_autoplace no)
+			(effects
+				(font
+					(size 1.27 1.27)
+				)
+				(justify left bottom)
+			)
+		)
+		(property "Sheetfile" "Interface.kicad_sch"
+			(at 125.73 105.9946 0)
+			(show_name no)
+			(do_not_autoplace no)
+			(effects
+				(font
+					(size 1.27 1.27)
+				)
+				(justify left top)
+			)
+		)
+		(instances
+			(project "echoear_coreboard"
+				(path "/919b249b-28e6-49d6-a46c-47b0cfe0d5d1"
+					(page "3")
+				)
+			)
+		)
+	)
+	(sheet
+		(at 71.12 92.71)
+		(size 24.13 12.7)
+		(exclude_from_sim no)
+		(in_bom yes)
+		(on_board yes)
+		(dnp no)
+		(fields_autoplaced yes)
+		(stroke
+			(width 0.1524)
+			(type solid)
+		)
+		(fill
+			(color 0 0 0 0)
+		)
+		(property "Sheetname" "MCU"
+			(at 71.12 91.9984 0)
+			(show_name no)
+			(do_not_autoplace no)
+			(effects
+				(font
+					(size 1.27 1.27)
+				)
+				(justify left bottom)
+			)
+		)
+		(property "Sheetfile" "MCU.kicad_sch"
+			(at 71.12 105.9946 0)
+			(show_name no)
+			(do_not_autoplace no)
+			(effects
+				(font
+					(size 1.27 1.27)
+				)
+				(justify left top)
+			)
+		)
+		(instances
+			(project "echoear_coreboard"
+				(path "/919b249b-28e6-49d6-a46c-47b0cfe0d5d1"
+					(page "2")
+				)
+			)
+		)
+	)
 	(sheet_instances
 		(path "/"

Commit message: Finished coreboard SCH w/o ERC check
Other:
- added sheet codec1 (codec1.kicad_sch)
Changed lines of the file:
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@@
 	)
 	(sheet
-		(at 185.42 92.71)
+		(at 161.29 91.44)
 		(size 26.67 13.97)
 		(exclude_from_sim no)
@@
 		)
 		(property "Sheetname" "codec"
-			(at 185.42 91.9984 0)
+			(at 161.29 90.7284 0)
 			(show_name no)
 			(do_not_autoplace no)
@@
 		)
 		(property "Sheetfile" "codec.kicad_sch"
-			(at 185.42 107.2646 0)
+			(at 161.29 105.9946 0)
 			(show_name no)
 			(do_not_autoplace no)
@@
 	)
 	(sheet
-		(at 125.73 91.44)
+		(at 101.6 90.17)
 		(size 24.13 13.97)
 		(exclude_from_sim no)
@@
 		)
 		(property "Sheetname" "Interface"
-			(at 125.73 90.7284 0)
+			(at 101.6 89.4584 0)
 			(show_name no)
 			(do_not_autoplace no)
@@
 		)
 		(property "Sheetfile" "Interface.kicad_sch"
-			(at 125.73 105.9946 0)
+			(at 101.6 104.7246 0)
 			(show_name no)
 			(do_not_autoplace no)
@@
 	)
 	(sheet
-		(at 71.12 92.71)
+		(at 46.99 91.44)
 		(size 24.13 12.7)
 		(exclude_from_sim no)
@@
 		)
 		(property "Sheetname" "MCU"
-			(at 71.12 91.9984 0)
+			(at 46.99 90.7284 0)
 			(show_name no)
 			(do_not_autoplace no)
@@
 		)
 		(property "Sheetfile" "MCU.kicad_sch"
-			(at 71.12 105.9946 0)
+			(at 46.99 104.7246 0)
 			(show_name no)
 			(do_not_autoplace no)
@@
 				)
 			)
+		)
+	)
+	(sheet
+		(at 213.36 91.44)
+		(size 26.67 13.97)
+		(exclude_from_sim no)
+		(in_bom yes)
+		(on_board yes)
+		(dnp no)
+		(fields_autoplaced yes)
+		(stroke
+			(width 0.1524)
+			(type solid)
+		)
+		(fill
+			(color 0 0 0 0)
+		)
+		(property "Sheetname" "codec1"
+			(at 213.36 90.7284 0)
+			(show_name no)
+			(do_not_autoplace no)
+			(effects
+				(font
+					(size 1.27 1.27)
+				)
+				(justify left bottom)
+			)
+		)
+		(property "Sheetfile" "codec1.kicad_sch"
+			(at 213.36 105.9946 0)
+			(show_name no)
+			(do_not_autoplace no)
+			(effects
+				(font
+					(size 1.27 1.27)
+				)
+				(justify left top)
+			)
+		)
+		(instances
+			(project "echoear_coreboard"
+				(path "/919b249b-28e6-49d6-a46c-47b0cfe0d5d1"
+					(page "5")
+				)
+			)
