File: echoear_coreboard/echoear_coreboard.kicad_pcb (KiCad board)
At the start: 4 copper layers, 44 x 27.2 mm, 88 parts, among them CN1 HC-1.25-2PLT, CN2 HC-1.25-2PLT, CN3 YXT-BB10-24S-02, CN4 HC-1.25-2PLT, Q1 AO3401A, Q2 AO3400A, Q3 LBSS138DW1T1G, Q4 LBSS138DW1T1G, U1 ESP32-S3-WROOM-1, U2 8.03A0.039200, U3 BMI270, U4 XC6206P332MR, U6 ES8311, U7 NS4150, U8 ES7210

Commit message: Front CU PCB placed
Parts:
- moved CN3 114.0 mm to (152.5, 98.9)
- moved U2 100.8 mm to (141.4, 96.6)
- moved FPC1 82.5 mm to (122.0, 91.2), turned to 100 degrees
- moved FPC2 67.5 mm to (129.1, 96.2)
- moved CN4 56.7 mm to (123.8, 81.9), turned to -110 degrees
- moved U3 2.76 mm to (47.6, 92.7)
Routing:
- net unconnected-(U2-Pad24): vias 0 -> 1
- net GND: vias 0 -> 4
- net /codec1/VOP: vias 0 -> 1
- net /codec1/ADC_MICBIAS12: vias 0 -> 1
- net /codec1/ADC_MIC2_N: vias 0 -> 1
- net /Interface/TP_INT: vias 0 -> 1
- net /Interface/MCU_3V3: vias 0 -> 1
- net (no net): vias 261 -> 251

Commit message: Arranging of Fu Cu
Parts:
- removed H2: ZX-PZ1.27-2-4PWZ, easyeda2kicad:HDR-SMD_8P-P1.27-LS5.5_ZX-PZ1.27-2-4PWZ
- added ?: , , F.Cu at (160.8, 82.0)
- added ?: , , F.Cu at (161.5, 84.4)
- added ?: , , F.Cu at (159.9, 79.6)
- added REF**: 1.5mm_pad, Library:1.5mm_pad, F.Cu at (157.2, 70.9)
- added REF**: 1.5mm_pad, Library:1.5mm_pad, F.Cu at (124.5, 72.1)
- added REF**: 1.5mm_pad, Library:1.5mm_pad, F.Cu at (158.7, 73.0)
- renumbered FPC2 to MIC
Routing:
- net GND: track 0.00 -> 7.42 mm, vias 4 -> 108
- net unconnected-(U2-Pad24): vias 1 -> 0
- net GNDA: vias 0 -> 8
- net /codec1/MCU_3V3: vias 0 -> 1
- net /codec1/LED_G: vias 0 -> 1
- net /codec1/ADC_MIC2_P: vias 0 -> 1
- net /codec1/ADC_MIC1_P: vias 0 -> 1
- net /codec1/ADC_MIC1_N: vias 0 -> 1
- net /codec/MCU_3V3: vias 0 -> 1
- net /codec/CODEC_3V3: vias 0 -> 4
- net /MCU/TP_INT: vias 0 -> 1
- net /MCU/POWER_CTRL: vias 0 -> 1
- net /MCU/PA_CTRL: vias 0 -> 1
- net /MCU/MCU_3V3: vias 0 -> 2
- net /MCU/LED_G: vias 0 -> 3
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